Commit message: make gazebo+moveit work on ur10

File: raw3-6/calibration/calibration_offset.urdf.xacro (robot description, xacro)
@@ -1,38 +1,45 @@
 <?xml version="1.0" ?>
-<robot>
+<robot xmlns:xacro="http://www.ros.org/wiki/xacro">
 	<!-- ***************** -->
 	<!-- base calibration -->
 	<!-- ***************** -->
 	<!-- laser front mount positions | relative to base_link -->
-	<property name="offset_laser_front_x" value="0.0"/>
-	<property name="offset_laser_front_y" value="0.0"/>
-	<property name="offset_laser_front_z" value="0.0"/>
-	<property name="offset_laser_front_roll" value="${M_PI}"/>
-	<property name="offset_laser_front_pitch" value="0.0"/>
-	<property name="offset_laser_front_yaw" value="0.0"/>
+	<xacro:property name="offset_laser_front_x" value="0.0"/>
+	<xacro:property name="offset_laser_front_y" value="0.0"/>
+	<xacro:property name="offset_laser_front_z" value="0.0"/>
+	<xacro:property name="offset_laser_front_roll" value="0.0"/>
+	<xacro:property name="offset_laser_front_pitch" value="0.0"/>
+	<xacro:property name="offset_laser_front_yaw" value="0.0"/>
 	<!-- laser rear mount positions | relative to base_link -->
-	<property name="offset_laser_rear_x" value="0.0"/>
-	<property name="offset_laser_rear_y" value="0.0"/>
-	<property name="offset_laser_rear_z" value="0.0"/>
-	<property name="offset_laser_rear_roll" value="0.0"/>
-	<property name="offset_laser_rear_pitch" value="${-M_PI}"/>
-	<property name="offset_laser_rear_yaw" value="${M_PI}"/>
-	<!-- *********************************** -->
-	<!-- kinematic chain reference positions -->
-	<!-- *********************************** -->
-	<!-- this feature is no longer supported as urdfdom does not parse the according 'calibration_rising' tag -->
+	<xacro:property name="offset_laser_rear_x" value="0.0"/>
+	<xacro:property name="offset_laser_rear_y" value="0.0"/>
+	<xacro:property name="offset_laser_rear_z" value="0.0"/>
+	<xacro:property name="offset_laser_rear_roll" value="0.0"/>
+	<xacro:property name="offset_laser_rear_pitch" value="0.0"/>
+	<xacro:property name="offset_laser_rear_yaw" value="0.0"/>
+	<!-- *********************** -->
+	<!-- upper robot calibration -->
+	<!-- *********************** -->
 	<!-- tower mount positions | relative to base_link -->
-	<property name="offset_tower_x" value="0.0"/>
-	<property name="offset_tower_y" value="0.0"/>
-	<property name="offset_tower_z" value="0.0"/>
-	<property name="offset_tower_roll" value="0.0"/>
-	<property name="offset_tower_pitch" value="0.0"/>
-	<property name="offset_tower_yaw" value="0.0"/>
+	<xacro:property name="offset_tower_x" value="0.0"/>
+	<xacro:property name="offset_tower_y" value="0.0"/>
+	<xacro:property name="offset_tower_z" value="0.0"/>
+	<xacro:property name="offset_tower_roll" value="0.0"/>
+	<xacro:property name="offset_tower_pitch" value="0.0"/>
+	<xacro:property name="offset_tower_yaw" value="0.0"/>
 	<!-- arm mount positions | relative to base_link -->
-	<property name="offset_arm_x" value="0.0"/>
-	<property name="offset_arm_y" value="0.0"/>
-	<property name="offset_arm_z" value="0.0"/>
-	<property name="offset_arm_roll" value="0.0"/>
-	<property name="offset_arm_pitch" value="0.0"/>
-	<property name="offset_arm_yaw" value="0.0"/>
+	<xacro:property name="offset_arm_x" value="0.0"/>
+	<xacro:property name="offset_arm_y" value="0.0"/>
+	<xacro:property name="offset_arm_z" value="0.0"/>
+	<xacro:property name="offset_arm_roll" value="0.0"/>
+	<xacro:property name="offset_arm_pitch" value="0.0"/>
+	<xacro:property name="offset_arm_yaw" value="0.0"/>
+	<!-- gripper mount positions | relative to arm_ee_link -->
+    <!--directly defined at ./src/cob_robots/cob_hardware_config/robots/raw3-6/urdf/raw3-6.urdf.xacro-->
+	<!--<xacro:property name="offset_gripper_x" value="0.0"/>-->
+	<!--<xacro:property name="offset_gripper_y" value="0.0"/>-->
+	<!--<xacro:property name="offset_gripper_z" value="0.0"/>-->
+	<!--<xacro:property name="offset_gripper_roll" value="0.0"/>-->
+	<!--<xacro:property name="offset_gripper_pitch" value="0.0"/>-->
+	<!--<xacro:property name="offset_gripper_yaw" value="0.0"/>-->
 </robot>
